File: kicad/nand-test.kicad_pcb (KiCad board)
At the start: 2 copper layers, 48.3 x 33 mm, 9 parts, among them J1 PWR, Q1 2N3904, Q2 2N3904, SW1 SW_SPST, SW2 SW_SPST

Commit message: generated gerber and gcode
Changed lines of the file:
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@@
     (aux_axis_origin 81.28 55.88)
     (pcbplotparams
-      (layerselection 0x00010fc_ffffffff)
+      (layerselection 0x0001000_fffffffe)
       (disableapertmacros false)
       (usegerberextensions false)
@@
       (viasonmask false)
       (mode 1)
-      (useauxorigin false)
+      (useauxorigin true)
       (hpglpennumber 1)
       (hpglpenspeed 20)
@@
       (outputformat 1)
       (mirror false)
-      (drillshape 1)
+      (drillshape 0)
       (scaleselection 1)
-      (outputdirectory "")
+      (outputdirectory "../gerber/")
     )
   )
@@
     (fp_arc (start -0.483625 1.753625) (mid -1.021221 -0.949055) (end 1.27 -2.48) (layer "F.Fab") (width 0.1))
     (fp_arc (start 1.27 -2.48) (mid 3.561221 -0.949055) (end 3.023625 1.753625) (layer "F.Fab") (width 0.1))
-    (pad "1" thru_hole rect (at -1 0 180) (size 1.05 1.5) (drill 0.75) (layers *.Cu *.Mask)
+    (pad "1" thru_hole rect (at -1 0 180) (size 1.05 1.5) (drill 0.8) (layers *.Cu *.Mask)
       (net 1 "GND") (pinfunction "E") (pintype "passive"))
-    (pad "2" thru_hole oval (at 1.27 0 180) (size 1.05 1.5) (drill 0.75) (layers *.Cu *.Mask)
+    (pad "2" thru_hole oval (at 1.27 0 180) (size 1.05 1.5) (drill 0.8) (layers *.Cu *.Mask)
       (net 6 "Net-(Q2-Pad2)") (pinfunction "B") (pintype "passive"))
-    (pad "3" thru_hole oval (at 3.5 0 180) (size 1.05 1.5) (drill 0.75) (layers *.Cu *.Mask)
+    (pad "3" thru_hole oval (at 3.5 0 180) (size 1.05 1.5) (drill 0.8) (layers *.Cu *.Mask)
       (net 4 "Net-(Q1-Pad1)") (pinfunction "C") (pintype "passive"))
     (model "${KICAD6_3DMODEL_DIR}/Package_TO_SOT_THT.3dshapes/TO-92_Inline.wrl"
@@
     (fp_arc (start -1.23 -1.469694) (mid 4.17 0.000016) (end -1.230016 1.469666) (layer "F.Fab") (width 0.1))
     (fp_circle (center 1.27 0) (end 3.77 0) (layer "F.Fab") (width 0.1) (fill none))
-    (pad "1" thru_hole rect (at 0 0 90) (size 1.8 1.8) (drill 0.9) (layers *.Cu *.Mask)
+    (pad "1" thru_hole rect (at 0 0 90) (size 1.8 1.8) (drill 0.8) (layers *.Cu *.Mask)
       (net 1 "GND") (pinfunction "K") (pintype "passive"))
-    (pad "2" thru_hole circle (at 2.54 0 90) (size 1.8 1.8) (drill 0.9) (layers *.Cu *.Mask)
+    (pad "2" thru_hole circle (at 2.54 0 90) (size 1.8 1.8) (drill 0.8) (layers *.Cu *.Mask)
       (net 2 "Net-(D1-Pad2)") (pinfunction "A") (pintype "passive"))
     (model "${KICAD6_3DMODEL_DIR}/LED_THT.3dshapes/LED_D5.0mm.wrl"
@@
     (fp_arc (start 1.27 -2.48) (mid 3.561221 -0.949055) (end 3.023625 1.753625) (layer "F.Fab") (width 0.1))
     (fp_arc (start -0.483625 1.753625) (mid -1.021221 -0.949055) (end 1.27 -2.48) (layer "F.Fab") (width 0.1))
-    (pad "1" thru_hole rect (at -1 0 180) (size 1.05 1.5) (drill 0.75) (layers *.Cu *.Mask)
+    (pad "1" thru_hole rect (at -1 0 180) (size 1.05 1.5) (drill 0.8) (layers *.Cu *.Mask)
       (net 4 "Net-(Q1-Pad1)") (pinfunction "E") (pintype "passive"))
-    (pad "2" thru_hole oval (at 1.27 0 180) (size 1.05 1.5) (drill 0.75) (layers *.Cu *.Mask)
+    (pad "2" thru_hole oval (at 1.27 0 180) (size 1.05 1.5) (drill 0.8) (layers *.Cu *.Mask)
       (net 5 "Net-(Q1-Pad2)") (pinfunction "B") (pintype "passive"))
-    (pad "3" thru_hole oval (at 3.5 0 180) (size 1.05 1.5) (drill 0.75) (layers *.Cu *.Mask)
+    (pad "3" thru_hole oval (at 3.5 0 180) (size 1.05 1.5) (drill 0.8) (layers *.Cu *.Mask)
       (net 2 "Net-(D1-Pad2)") (pinfunction "C") (pintype "passive"))
     (model "${KICAD6_3DMODEL_DIR}/Package_TO_SOT_THT.3dshapes/TO-92_Inline.wrl"
@@
     (fp_line (start 6.25 -0.75) (end 6.25 5.25) (layer "F.Fab") (width 0.1))
     (fp_circle (center 3.25 2.25) (end 1.25 2.5) (layer "F.Fab") (width 0.1) (fill none))
-    (pad "1" thru_hole circle (at 6.5 0 90) (size 2 2) (drill 1.1) (layers *.Cu *.Mask)
+    (pad "1" thru_hole circle (at 6.5 0 90) (size 2 2) (drill 0.8) (layers *.Cu *.Mask)
       (net 3 "+5V") (pinfunction "A") (pintype "passive"))
-    (pad "1" thru_hole circle (at 0 0 90) (size 2 2) (drill 1.1) (layers *.Cu *.Mask)
+    (pad "1" thru_hole circle (at 0 0 90) (size 2 2) (drill 0.8) (layers *.Cu *.Mask)
       (net 3 "+5V") (pinfunction "A") (pintype "passive"))
-    (pad "2" thru_hole circle (at 0 4.5 90) (size 2 2) (drill 1.1) (layers *.Cu *.Mask)
+    (pad "2" thru_hole circle (at 0 4.5 90) (size 2 2) (drill 0.8) (layers *.Cu *.Mask)
       (net 7 "Net-(R1-Pad1)") (pinfunction "B") (pintype "passive"))
-    (pad "2" thru_hole circle (at 6.5 4.5 90) (size 2 2) (drill 1.1) (layers *.Cu *.Mask)
+    (pad "2" thru_hole circle (at 6.5 4.5 90) (size 2 2) (drill 0.8) (layers *.Cu *.Mask)
       (net 7 "Net-(R1-Pad1)") (pinfunction "B") (pintype "passive"))
     (model "${KICAD6_3DMODEL_DIR}/Button_Switch_THT.3dshapes/SW_PUSH_6mm.wrl"
@@
     (fp_line (start 6.25 5.25) (end 0.25 5.25) (layer "F.Fab") (width 0.1))
     (fp_circle (center 3.25 2.25) (end 1.25 2.5) (layer "F.Fab") (width 0.1) (fill none))
-    (pad "1" thru_hole circle (at 0 0 90) (size 2 2) (drill 1.1) (layers *.Cu *.Mask)
+    (pad "1" thru_hole circle (at 0 0 90) (size 2 2) (drill 0.8) (layers *.Cu *.Mask)
       (net 3 "+5V") (pinfunction "A") (pintype "passive"))
-    (pad "1" thru_hole circle (at 6.5 0 90) (size 2 2) (drill 1.1) (layers *.Cu *.Mask)
+    (pad "1" thru_hole circle (at 6.5 0 90) (size 2 2) (drill 0.8) (layers *.Cu *.Mask)
       (net 3 "+5V") (pinfunction "A") (pintype "passive"))
-    (pad "2" thru_hole circle (at 0 4.5 90) (size 2 2) (drill 1.1) (layers *.Cu *.Mask)
+    (pad "2" thru_hole circle (at 0 4.5 90) (size 2 2) (drill 0.8) (layers *.Cu *.Mask)
       (net 8 "Net-(R2-Pad1)") (pinfunction "B") (pintype "passive"))
-    (pad "2" thru_hole circle (at 6.5 4.5 90) (size 2 2) (drill 1.1) (layers *.Cu *.Mask)
+    (pad "2" thru_hole circle (at 6.5 4.5 90) (size 2 2) (drill 0.8) (layers *.Cu *.Mask)
       (net 8 "Net-(R2-Pad1)") (pinfunction "B") (pintype "passive"))
     (model "${KICAD6_3DMODEL_DIR}/Button_Switch_THT.3dshapes/SW_PUSH_6mm.wrl"
@@
     (fp_arc (start 6.54 -5.05) (mid 6.715733 -4.551652) (end 6.485532 -4.076005) (layer "F.Fab") (width 0.1))
     (fp_arc (start 3.39 -5) (mid 4.949737 -5.764867) (end 6.538239 -5.061686) (layer "F.Fab") (width 0.1))
-    (pad "1" thru_hole rect (at 0 0 270) (size 1.98 3.96) (drill 1.32) (layers *.Cu *.Mask)
+    (pad ".8" thru_hole oval (at 5 0 270) (size 1.98 3.96) (drill 0.8) (layers *.Cu *.Mask)
+      (net 1 "GND") (pinfunction "Pin_2") (pintype "passive"))
+    (pad "1" thru_hole rect (at 0 0 270) (size 1.98 3.96) (drill 0.8) (layers *.Cu *.Mask)
       (net 3 "+5V") (pinfunction "Pin_1") (pintype "passive"))
-    (pad "2" thru_hole oval (at 5 0 270) (size 1.98 3.96) (drill 1.32) (layers *.Cu *.Mask)
-      (net 1 "GND") (pinfunction "Pin_2") (pintype "passive"))
     (model "${KICAD6_3DMODEL_DIR}/TerminalBlock.3dshapes/TerminalBlock_Altech_AK300-2_P5.00mm.wrl"
       (offset (xyz 0 0 0))
@@
     (effects (font (size 1 1) (thickness 0.15)))
   )
-  (dimension (type orthogonal) (layer "Edge.Cuts")
-    (pts (xy 81.28 55.88) (xy 81.28 88.9))
-    (height -5.08)
+  (dimension (type orthogonal) (layer "Dwgs.User")
+    (pts (xy 129.54 55.88) (xy 129.54 88.9))
+    (height 7.62)
     (orientation 1)
-    (gr_text "33.0200 mm" (at 75.05 72.39 90) (layer "Edge.Cuts")
+    (gr_text "33.0200 mm" (at 136.01 72.39 90) (layer "Dwgs.User")
       (effects (font (size 1 1) (thickness 0.15)))
     )
     (format (units 3) (units_format 1) (precision 4))
-    (style (thickness 0.1) (arrow_length 1.27) (text_position_mode 0) (extension_height 0.58642) (extension_offset 0.5) keep_text_aligned)
-  )
-  (dimension (type orthogonal) (layer "Edge.Cuts")
-    (pts (xy 129.54 55.88) (xy 81.28 55.88))
+    (style (thickness 0.15) (arrow_length 1.27) (text_position_mode 0) (extension_height 0.58642) (extension_offset 0.5) keep_text_aligned)
+  )
+  (dimension (type orthogonal) (layer "Dwgs.User")
+    (pts (xy 81.28 55.88) (xy 129.54 55.88))
     (height -3.81)
     (orientation 0)
-    (gr_text "48.2600 mm" (at 105.41 50.92) (layer "Edge.Cuts")
+    (gr_text "48.2600 mm" (at 105.41 50.92) (layer "Dwgs.User")
       (effects (font (size 1 1) (thickness 0.15)))
     )
     (format (units 3) (units_format 1) (precision 4))
-    (style (thickness 0.1) (arrow_length 1.27) (text_position_mode 0) (extension_height 0.58642) (extension_offset 0.5) keep_text_aligned)
+    (style (thickness 0.15) (arrow_length 1.27) (text_position_mode 0) (extension_height 0.58642) (extension_offset 0.5) keep_text_aligned)
   )
   (segment (start 105.33 83.74) (end 105.41 83.82) (width 0.5) (layer "B.Cu") (net 1))
