File: kicad/nand-test.kicad_sch (KiCad schematic)
At the start: 9 parts, among them J1 PWR, Q1 2N3904, Q2 2N3904, SW1 SW_SPST, SW2 SW_SPST

Commit message: generated gerber and gcode
Other:
- title: (none) -> nand-pcb-test
Changed lines of the file:
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@@
 (kicad_sch (version 20211123) (generator eeschema)
   (paper "A4")
+  (title_block
+    (title "nand-pcb-test")
+    (comment 1 "Barrett Otte")
+    (comment 2 "https://github.com/barrettotte/nand-pcb-test")
+  )
   (junction (at 63.5 73.66) (diameter 0) (color 0 0 0 0)
   )
